Commit message: fixed

File: robots/sia5f_arm.urdf (robot description, URDF)
Before this commit: robot motoman_sia5f_arm, 9 links, 8 joints
Joints:
- joint joint_s: limit lower=${-180*deg} upper=${180*deg} effort=0 velocity=${200*deg} -> lower=${-180.0*deg} upper=${180.0*deg} effort=0 velocity=${200.0*deg}

Commit message: Fixed transformation

File: robots/sia5f_arm.urdf (robot description, URDF)
Before this commit: robot motoman_sia5f_arm, 9 links, 8 joints
Links:
- link base_link: mass 400 -> 9.23913043478
- link link_b: mass 2.3902999 -> 0.869565217391
- link link_e: mass 4.7092004 -> 1.30434782609
- link link_l: mass 5.227999 -> 7.60869565217
- link link_r: mass 3.0270943 -> 0.978260869565
- link link_s: mass 13.746057 -> 8.36956521739
- link link_t: mass 0.63670412 -> 0.54347826087
- link link_u: mass 3.1488649 -> 1.08695652174

Commit message: Fixed name

File: robots/sia5f_arm.urdf (robot description, URDF)
Before this commit: robot motoman_sia5f_arm, 9 links, 8 joints
Links:
- link base_link: geometry collision mesh filename=file://$(find yaskawa_description_ros2)/meshes/collision/ba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; visual mesh filename=file://$(find yaskawa_description_ros2)/meshes/visual/base.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
- link link_b: geometry collision mesh filename=file://$(find yaskawa_description_ros2)/meshes/collision/li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; visual mesh filename=file://$(find yaskawa_description_ros2)/meshes/visual/link_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
- link link_e: geometry collision mesh filename=file://$(find yaskawa_description_ros2)/meshes/collision/li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; visual mesh filename=file://$(find yaskawa_description_ros2)/meshes/visual/link_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
- link link_l: geometry collision mesh filename=file://$(find yaskawa_description_ros2)/meshes/collision/li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; visual mesh filename=file://$(find yaskawa_description_ros2)/meshes/visual/link_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
- link link_r: geometry collision mesh filename=file://$(find yaskawa_description_ros2)/meshes/collision/li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; visual mesh filename=file://$(find yaskawa_description_ros2)/meshes/visual/link_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
- link link_s: geometry collision mesh filename=file://$(find yaskawa_description_ros2)/meshes/collision/li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; visual mesh filename=file://$(find yaskawa_description_ros2)/meshes/visual/link_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
- link link_t: geometry collision mesh filename=file://$(find yaskawa_description_ros2)/meshes/collision/li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; visual mesh filename=file://$(find yaskawa_description_ros2)/meshes/visual/link_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
- link link_u: geometry collision mesh filename=file://$(find yaskawa_description_ros2)/meshes/collision/li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; visual mesh filename=file://$(find yaskawa_description_ros2)/meshes/visual/link_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

File: robots/sia5f_arm.xacro (robot description, xacro)
@@ -1,4 +1,4 @@
 <?xml version='1.0' encoding='utf-8'?>
 <robot xmlns:xacro="http://www.ros.org/wiki/xacro" name="motoman_sia5f">
-  <xacro:include filename="$(find yaskawa_description)/robots/sia5f_arm.urdf"/>
+  <xacro:include filename="$(find yaskawa_description_ros2)/robots/sia5f_arm.urdf"/>
 </robot>
